File: eagle/schematics/dimmer-aussen/untitled.brd (EAGLE design)
At the start: 100 x 80 mm, 6 parts, among them M3 ARDUINO-PRO-MINI-3.3V

Commit message: some changes
Parts:
- U$1: device cc1101:CC1101-MODULE-SMD -> cc1101:PFOSTEN
- moved U$1 5.24 mm to (88.9, 29.2)
Connections:
- net N$3: now also M3.J6.7; no longer M3.J6.12
Routing:
- net N$2: track 0.00 -> 33.3 mm
- net N$6: track 0.00 -> 12.5 mm
- net N$5: track 0.00 -> 7.90 mm
- net N$7: track 0.00 -> 7.46 mm
- net N$4: track 0.00 -> 7.30 mm
- net N$3: track 0.00 -> 7.23 mm
Changed lines of the file:
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@@
 <elements>
 <element name="M3" library="diy-modules" package="ARDUINO-PRO-MINI" value="ARDUINO-PRO-MINI-3.3V" x="81.28" y="22.86"/>
-<element name="U$1" library="cc1101" package="CC1101-MODULE-SMD" value="" x="90.17" y="24.13" rot="R270"/>
+<element name="U$1" library="cc1101" package="PFOSTEN" value="" x="88.9" y="29.21" rot="R270"/>
 <element name="T1" library="zetex" package="SOT-23" value="" x="72.39" y="7.62">
 <attribute name="MF" value="" x="72.39" y="7.62" size="1.778" layer="27" display="off"/>
@@
 <signal name="N$2">
 <contactref element="M3" pad="J6.2"/>
-<contactref element="U$1" pad="GND"/>
 <contactref element="M3" pad="J7.9"/>
 <contactref element="T1" pad="2"/>
-<wire x1="71.4502" y1="8.636" x2="94.67" y2="34.63" width="0" layer="19" extent="1-1"/>
-<wire x1="71.12" y1="30.48" x2="71.4502" y2="8.636" width="0" layer="19" extent="1-1"/>
+<contactref element="U$1" pad="GND"/>
+<wire x1="76.2" y1="15.24" x2="89.6664" y2="28.7064" width="0.4064" layer="1"/>
+<wire x1="95.3082" y1="29.04091875" x2="95.3082" y2="30.87908125" width="0.4064" layer="1"/>
+<wire x1="89.6664" y1="28.7064" x2="94.97368125" y2="28.7064" width="0.4064" layer="1"/>
+<wire x1="94.97368125" y1="28.7064" x2="95.3082" y2="29.04091875" width="0.4064" layer="1"/>
+<wire x1="93.4" y1="32.78728125" x2="93.4" y2="36.71" width="0.4064" layer="1"/>
+<wire x1="95.3082" y1="30.87908125" x2="93.4" y2="32.78728125" width="0.4064" layer="1"/>
 <wire x1="76.2" y1="15.24" x2="71.12" y2="30.48" width="0" layer="19" extent="1-1"/>
+<wire x1="71.4502" y1="8.636" x2="76.2" y2="15.24" width="0" layer="19" extent="1-1"/>
 </signal>
 <signal name="N$3">
-<contactref element="M3" pad="J6.12"/>
 <contactref element="U$1" pad="CSN"/>
-<wire x1="82.67" y1="34.63" x2="96.52" y2="30.48" width="0" layer="19" extent="1-1"/>
+<contactref element="M3" pad="J6.7"/>
+<wire x1="83.82" y1="30.48" x2="81.4" y2="32.9" width="0.4064" layer="1"/>
+<wire x1="81.4" y1="32.9" x2="81.4" y2="36.71" width="0.4064" layer="1"/>
 </signal>
 <signal name="N$4">
 <contactref element="M3" pad="J6.11"/>
 <contactref element="U$1" pad="SI"/>
-<wire x1="92.67" y1="34.63" x2="93.98" y2="30.48" width="0" layer="19" extent="1-1"/>
+<wire x1="93.98" y1="30.48" x2="91.4" y2="33.06" width="0.4064" layer="1"/>
+<wire x1="91.4" y1="33.06" x2="91.4" y2="36.71" width="0.4064" layer="1"/>
 </signal>
 <signal name="N$5">
 <contactref element="M3" pad="J6.10"/>
 <contactref element="U$1" pad="SO"/>
-<wire x1="88.67" y1="34.63" x2="91.44" y2="30.48" width="0" layer="19" extent="1-1"/>
+<wire x1="91.44" y1="30.48" x2="87.4" y2="34.52" width="0.4064" layer="1"/>
+<wire x1="87.4" y1="34.52" x2="87.4" y2="36.71" width="0.4064" layer="1"/>
 </signal>
 <signal name="N$6">
 <contactref element="M3" pad="J6.9"/>
 <contactref element="U$1" pad="SCLK"/>
-<wire x1="88.9" y1="30.48" x2="90.67" y2="34.63" width="0" layer="19" extent="1-1"/>
+<wire x1="90.9586" y1="29.3178" x2="91.9214" y2="29.3178" width="0.4064" layer="1"/>
+<wire x1="91.9214" y1="29.3178" x2="92.6022" y2="29.9986" width="0.4064" layer="1"/>
+<wire x1="92.6022" y1="29.9986" x2="92.6022" y2="30.9614" width="0.4064" layer="1"/>
+<wire x1="88.9" y1="30.48" x2="89.7964" y2="30.48" width="0.4064" layer="1"/>
+<wire x1="89.4" y1="34.1636" x2="89.4" y2="36.71" width="0.4064" layer="1"/>
+<wire x1="89.7964" y1="30.48" x2="90.9586" y2="29.3178" width="0.4064" layer="1"/>
+<wire x1="92.6022" y1="30.9614" x2="89.4" y2="34.1636" width="0.4064" layer="1"/>
 </signal>
 <signal name="N$1">
@@
 <contactref element="X2" pad="1"/>
 <contactref element="X2" pad="2"/>
-<wire x1="88.9" y1="4.445" x2="96.67" y2="34.63" width="0" layer="19" extent="1-1"/>
+<wire x1="88.9" y1="4.445" x2="95.4" y2="36.71" width="0" layer="19" extent="1-1"/>
 <wire x1="93.98" y1="4.445" x2="88.9" y2="4.445" width="0" layer="19" extent="1-1"/>
 <wire x1="76.2" y1="30.48" x2="93.98" y2="4.445" width="0" layer="19" extent="1-1"/>
@@
 <contactref element="U$1" pad="GDO0"/>
 <contactref element="M3" pad="J6.8"/>
-<wire x1="86.36" y1="30.48" x2="84.67" y2="34.63" width="0" layer="19" extent="1-1"/>
+<wire x1="86.36" y1="30.48" x2="83.4" y2="33.44" width="0.4064" layer="1"/>
+<wire x1="83.4" y1="33.44" x2="83.4" y2="36.71" width="0.4064" layer="1"/>
 </signal>
 <signal name="N$8">
