File: eagle/schematics/dimmer-aussen/untitled.sch (EAGLE design)
At the start: 6 parts, among them M3 ARDUINO-PRO-MINI-3.3V

Commit message: some changes
Parts:
- U$1: device cc1101:CC1101-MODULESMD -> cc1101:CC1101-MODULEPFOSTEN
Connections:
- net N$3: now also M3.A1(PC1,ADC1); no longer M3.D10(PB2,SS)
